File: Layout/Processor/Power.sch (KiCad schematic (older format))
At the start: 9 parts, among them U11 LM1085-5.0, U5 AP2112K-3.3

Commit message: Adjust layouts
Connections:
- net labels added: 3.3V, 5V
- net labels removed: +3.3V, +5V
- wire segments 30 -> 29
