File: Cell/Layout/Processor/CommSelect.sch (KiCad schematic (older format))
At the start: 6 parts, among them U10 74LVC1G125, U2 74LVC1G125, U4 74LVC1G125, U7 74LVC1G125, U8 74LVC1G125, U9 74LVC1G125

Commit message: Do the processor board layout
Parts:
- renumbered U2 to U3, U7 to U5, U8 to U6, U9 to U7, U10 to U8
Changed lines of the file:
@@
 $EndDescr
 $Comp
-L 74xGxx:74LVC1G125 U2
+L 74xGxx:74LVC1G125 U3
 U 1 1 5FA68D2C
 P 3550 3000
-F 0 "U2" V 3571 2870 50  0000 R CNN
+F 0 "U3" V 3571 2870 50  0000 R CNN
 F 1 "74LVC1G125" V 3480 2870 50  0000 R CNN
 F 2 "Package_TO_SOT_SMD:SOT-353_SC-70-5_Handsoldering" H 3550 3000 50  0001 C CNN
@@
 	4350 3600 4350 3300
 $Comp
-L 74xGxx:74LVC1G125 U7
+L 74xGxx:74LVC1G125 U5
 U 1 1 5FA71EA0
 P 5150 3000
-F 0 "U7" V 5171 2870 50  0000 R CNN
+F 0 "U5" V 5171 2870 50  0000 R CNN
 F 1 "74LVC1G125" V 5080 2870 50  0000 R CNN
 F 2 "Package_TO_SOT_SMD:SOT-353_SC-70-5_Handsoldering" H 5150 3000 50  0001 C CNN
@@
 $EndComp
 $Comp
-L 74xGxx:74LVC1G125 U8
+L 74xGxx:74LVC1G125 U6
 U 1 1 5FA71EA6
 P 6000 3250
-F 0 "U8" V 5929 3121 50  0000 R CNN
+F 0 "U6" V 5929 3121 50  0000 R CNN
 F 1 "74LVC1G125" V 6020 3121 50  0000 R CNN
 F 2 "Package_TO_SOT_SMD:SOT-353_SC-70-5_Handsoldering" H 6000 3250 50  0001 C CNN
@@
 	5950 3600 5950 3300
 $Comp
-L 74xGxx:74LVC1G125 U9
+L 74xGxx:74LVC1G125 U7
 U 1 1 5FA738D8
 P 6750 3000
-F 0 "U9" V 6771 2870 50  0000 R CNN
+F 0 "U7" V 6771 2870 50  0000 R CNN
 F 1 "74LVC1G125" V 6680 2870 50  0000 R CNN
 F 2 "Package_TO_SOT_SMD:SOT-353_SC-70-5_Handsoldering" H 6750 3000 50  0001 C CNN
@@
 $EndComp
 $Comp
-L 74xGxx:74LVC1G125 U10
+L 74xGxx:74LVC1G125 U8
 U 1 1 5FA738DE
 P 7600 3250
-F 0 "U10" V 7529 3121 50  0000 R CNN
+F 0 "U8" V 7529 3121 50  0000 R CNN
 F 1 "74LVC1G125" V 7620 3121 50  0000 R CNN
 F 2 "Package_TO_SOT_SMD:SOT-353_SC-70-5_Handsoldering" H 7600 3250 50  0001 C CNN
@@
 	6550 3000 6550 2300
 $Comp
-L SparkFun-PowerSymbols:GND #GND0103
+L SparkFun-PowerSymbols:GND #GND08
 U 1 1 5FA78EEB
 P 7550 3600
-F 0 "#GND0103" H 7600 3550 45  0001 L BNN
+F 0 "#GND08" H 7600 3550 45  0001 L BNN
 F 1 "GND" H 7550 3430 45  0000 C CNN
 F 2 "" H 7550 3500 60  0001 C CNN
@@
 Connection ~ 7550 3600
 $Comp
-L SparkFun-PowerSymbols:3.3V #SUPPLY0103
+L SparkFun-PowerSymbols:3.3V #SUPPLY08
 U 1 1 5FA7978D
 P 7900 2650
-F 0 "#SUPPLY0103" H 7950 2650 45  0001 L BNN
+F 0 "#SUPPLY08" H 7950 2650 45  0001 L BNN
 F 1 "3.3V" H 7900 2926 45  0000 C CNN
 F 2 "XXX-00000" H 7900 2831 60  0000 C CNN
