File: Cell/Layout/Processor/Memory.sch (KiCad schematic (older format))
At the start: 1 part, among them U3 MB85RC256

Commit message: Do the processor board layout
Parts:
- renumbered U3 to U9
Changed lines of the file:
@@
 $EndDescr
 $Comp
-L Memory_NVRAM:FM24C64B U3
+L Memory_NVRAM:FM24C64B U9
 U 1 1 5F398A90
 P 5550 3550
-F 0 "U3" H 5550 4131 50  0000 C CNN
+F 0 "U9" H 5550 4131 50  0000 C CNN
 F 1 "MB85RC256" H 5550 4040 50  0000 C CNN
 F 2 "Package_SO:SOIC-8_3.9x4.9mm_P1.27mm" H 5550 3550 50  0001 C CNN
@@
 SCL
 $Comp
-L power:GND #PWR0119
+L power:GND #PWR03
 U 1 1 5F3990BA
 P 5550 4050
-F 0 "#PWR0119" H 5550 3800 50  0001 C CNN
+F 0 "#PWR03" H 5550 3800 50  0001 C CNN
 F 1 "GND" H 5555 3877 50  0000 C CNN
 F 2 "" H 5550 4050 50  0001 C CNN
@@
 Connection ~ 5550 3950
 $Comp
-L SparkFun-PowerSymbols:3.3V #SUPPLY0110
+L SparkFun-PowerSymbols:3.3V #SUPPLY09
 U 1 1 5FA7A40B
 P 5550 2900
-F 0 "#SUPPLY0110" H 5600 2900 45  0001 L BNN
+F 0 "#SUPPLY09" H 5600 2900 45  0001 L BNN
 F 1 "3.3V" H 5550 3176 45  0000 C CNN
 F 2 "XXX-00000" H 5550 3081 60  0000 C CNN
