File: Cell/Layout/Processor/Power.sch (KiCad schematic (older format))
At the start: 9 parts, among them U11 LM1085-5.0, U5 AP2112K-3.3

Commit message: Do the processor board layout
Parts:
- removed D1: DF02M, Diode_THT:Diode_Bridge_DIP-4_W7.62mm_P5.08mm, symbol Diode_Bridge:DF02M
- added CR1: DF01S, df01s:DF01S, symbol df01s:DF01S
- renumbered C7 to C1, C8 to C2, C9 to C3, C10 to C4, C11 to C5, C1 to C6, U11 to U10, U5 to U11
Connections:
- net +VDC: now also CR1.1 (+)
- net GND: now also CR1.2 (-)
- net PRI_HI: now also CR1.4 (AC2)
- net PRI_LO: now also CR1.3 (AC1)
Changed lines of the file:
@@
 $EndDescr
 $Comp
-L power:GND #PWR0121
+L power:GND #PWR05
 U 1 1 5F36338B
-P 2100 3450
-F 0 "#PWR0121" H 2100 3200 50  0001 C CNN
-F 1 "GND" H 2105 3277 50  0000 C CNN
-F 2 "" H 2100 3450 50  0001 C CNN
-F 3 "" H 2100 3450 50  0001 C CNN
-	1    2100 3450
-	1    0    0    -1
-$EndComp
-$Comp
-L power:PRI_HI #PWR0122
+P 1550 3750
+F 0 "#PWR05" H 1550 3500 50  0001 C CNN
+F 1 "GND" H 1555 3577 50  0000 C CNN
+F 2 "" H 1550 3750 50  0001 C CNN
+F 3 "" H 1550 3750 50  0001 C CNN
+	1    1550 3750
+	1    0    0    -1
+$EndComp
+$Comp
+L power:PRI_HI #PWR06
 U 1 1 5F363BA1
-P 2650 3000
-F 0 "#PWR0122" H 2650 2850 50  0001 C CNN
-F 1 "PRI_HI" H 2665 3173 50  0000 C CNN
-F 2 "" H 2650 3000 50  0001 C CNN
-F 3 "" H 2650 3000 50  0001 C CNN
-	1    2650 3000
-	1    0    0    -1
-$EndComp
-$Comp
-L power:+VDC #PWR0124
+P 3550 3250
+F 0 "#PWR06" H 3550 3100 50  0001 C CNN
+F 1 "PRI_HI" H 3565 3423 50  0000 C CNN
+F 2 "" H 3550 3250 50  0001 C CNN
+F 3 "" H 3550 3250 50  0001 C CNN
+	1    3550 3250
+	1    0    0    -1
+$EndComp
+$Comp
+L power:+VDC #PWR04
 U 1 1 5F364724
-P 3350 3450
-F 0 "#PWR0124" H 3350 3350 50  0001 C CNN
-F 1 "+VDC" H 3350 3725 50  0000 C CNN
-F 2 "" H 3350 3450 50  0001 C CNN
-F 3 "" H 3350 3450 50  0001 C CNN
-	1    3350 3450
-	1    0    0    -1
-$EndComp
-$Comp
-L power:+VDC #PWR0125
+P 1550 3300
+F 0 "#PWR04" H 1550 3200 50  0001 C CNN
+F 1 "+VDC" H 1550 3575 50  0000 C CNN
+F 2 "" H 1550 3300 50  0001 C CNN
+F 3 "" H 1550 3300 50  0001 C CNN
+	1    1550 3300
+	1    0    0    -1
+$EndComp
+$Comp
+L power:+VDC #PWR08
 U 1 1 5F36782D
 P 4950 3150
-F 0 "#PWR0125" H 4950 3050 50  0001 C CNN
+F 0 "#PWR08" H 4950 3050 50  0001 C CNN
 F 1 "+VDC" H 4950 3425 50  0000 C CNN
 F 2 "" H 4950 3150 50  0001 C CNN
@@
 $EndComp
 $Comp
-L Device:C C7
+L Device:C C1
 U 1 1 5F368CA1
 P 4550 3450
-F 0 "C7" H 4665 3496 50  0000 L CNN
+F 0 "C1" H 4665 3496 50  0000 L CNN
 F 1 "10u" H 4665 3405 50  0000 L CNN
 F 2 "Capacitor_SMD:C_0603_1608Metric_Pad1.05x0.95mm_HandSolder" H 4588 3300 50  0001 C CNN
@@
 $EndComp
 $Comp
-L Device:C C8
+L Device:C C2
 U 1 1 5F368F24
 P 4950 3450
-F 0 "C8" H 5065 3496 50  0000 L CNN
+F 0 "C2" H 5065 3496 50  0000 L CNN
 F 1 "1u" H 5065 3405 50  0000 L CNN
 F 2 "Capacitor_SMD:C_0603_1608Metric_Pad1.05x0.95mm_HandSolder" H 4988 3300 50  0001 C CNN
@@
 $EndComp
 $Comp
-L Device:C C9
+L Device:C C3
 U 1 1 5F3693E0
 P 5350 3450
-F 0 "C9" H 5465 3496 50  0000 L CNN
+F 0 "C3" H 5465 3496 50  0000 L CNN
 F 1 "0.1u" H 5465 3405 50  0000 L CNN
 F 2 "Capacitor_SMD:C_0603_1608Metric_Pad1.05x0.95mm_HandSolder" H 5388 3300 50  0001 C CNN
@@
 Connection ~ 4950 3600
 $Comp
-L power:GND #PWR0126
+L power:GND #PWR09
 U 1 1 5F36AFC7
 P 4950 3850
-F 0 "#PWR0126" H 4950 3600 50  0001 C CNN
+F 0 "#PWR09" H 4950 3600 50  0001 C CNN
 F 1 "GND" H 4955 3677 50  0000 C CNN
 F 2 "" H 4950 3850 50  0001 C CNN
@@
 $EndComp
 $Comp
-L Regulator_Linear:AP2112K-3.3 U5
+L Regulator_Linear:AP2112K-3.3 U11
 U 1 1 5F388344
 P 8400 3500
-F 0 "U5" H 8400 3842 50  0000 C CNN
+F 0 "U11" H 8400 3842 50  0000 C CNN
 F 1 "AP2112K-3.3" H 8400 3751 50  0000 C CNN
 F 2 "Package_TO_SOT_SMD:SOT-23-5" H 8400 3825 50  0001 C CNN
@@
 $EndComp
 $Comp
-L Device:C C10
+L Device:C C4
 U 1 1 5F38A05E
 P 7850 3850
-F 0 "C10" H 7965 3896 50  0000 L CNN
+F 0 "C4" H 7965 3896 50  0000 L CNN
 F 1 "0.1u" H 7965 3805 50  0000 L CNN
 F 2 "Capacitor_SMD:C_0603_1608Metric_Pad1.05x0.95mm_HandSolder" H 7888 3700 50  0001 C CNN
@@
 $EndComp
 $Comp
-L Device:C C11
+L Device:C C5
 U 1 1 5F38A758
 P 8950 3850
-F 0 "C11" H 9065 3896 50  0000 L CNN
+F 0 "C5" H 9065 3896 50  0000 L CNN
 F 1 "1u" H 9065 3805 50  0000 L CNN
 F 2 "Capacitor_SMD:C_0603_1608Metric_Pad1.05x0.95mm_HandSolder" H 8988 3700 50  0001 C CNN
@@
 	7850 3500 7850 3700
 $Comp
-L power:GND #PWR0132
+L power:GND #PWR011
 U 1 1 5F38E9E5
 P 8400 4000
-F 0 "#PWR0132" H 8400 3750 50  0001 C CNN
+F 0 "#PWR011" H 8400 3750 50  0001 C CNN
 F 1 "GND" H 8405 3827 50  0000 C CNN
 F 2 "" H 8400 4000 50  0001 C CNN
@@
 Connection ~ 8950 3400
 $Comp
-L Regulator_Linear:LM1085-5.0 U11
+L Regulator_Linear:LM1085-5.0 U10
 U 1 1 5FA399E2
 P 7100 3400
-F 0 "U11" H 7100 3642 50  0000 C CNN
+F 0 "U10" H 7100 3642 50  0000 C CNN
 F 1 "LM1085-5.0" H 7100 3551 50  0000 C CNN
 F 2 "Package_TO_SOT_SMD:TO-263-3_TabPin2" H 7100 3650 50  0001 C CIN
@@
 Connection ~ 7850 4000
 $Comp
-L power:+VDC #PWR0101
+L power:+VDC #PWR010
 U 1 1 5FA4F422
 P 6650 3200
-F 0 "#PWR0101" H 6650 3100 50  0001 C CNN
+F 0 "#PWR010" H 6650 3100 50  0001 C CNN
 F 1 "+VDC" H 6650 3475 50  0000 C CNN
 F 2 "" H 6650 3200 50  0001 C CNN
@@
 	6650 3400 6800 3400
 $Comp
-L Device:C C1
+L Device:C C6
 U 1 1 5FA607A6
 P 9450 3850
-F 0 "C1" H 9565 3896 50  0000 L CNN
+F 0 "C6" H 9565 3896 50  0000 L CNN
 F 1 "4.7u" H 9565 3805 50  0000 L CNN
 F 2 "Capacitor_SMD:C_0603_1608Metric_Pad1.05x0.95mm_HandSolder" H 9488 3700 50  0001 C CNN
@@
 Connection ~ 8950 4000
 $Comp
-L SparkFun-PowerSymbols:3.3V #SUPPLY0108
+L SparkFun-PowerSymbols:3.3V #SUPPLY011
 U 1 1 5FA792F6
 P 8950 3250
-F 0 "#SUPPLY0108" H 9000 3250 45  0001 L BNN
+F 0 "#SUPPLY011" H 9000 3250 45  0001 L BNN
 F 1 "3.3V" H 8950 3526 45  0000 C CNN
 F 2 "XXX-00000" H 8950 3431 60  0000 C CNN
@@
 $EndComp
 $Comp
-L SparkFun-PowerSymbols:5V #SUPPLY0109
+L SparkFun-PowerSymbols:5V #SUPPLY010
 U 1 1 5FA7984D
 P 7850 3250
-F 0 "#SUPPLY0109" H 7900 3250 45  0001 L BNN
+F 0 "#SUPPLY010" H 7900 3250 45  0001 L BNN
 F 1 "5V" H 7850 3526 45  0000 C CNN
 F 2 "XXX-00000" H 7850 3431 60  0000 C CNN
@@
 $EndComp
 $Comp
-L Diode_Bridge:DF02M D1
-U 1 1 5FA6EBE2
-P 2650 3450
-F 0 "D1" H 2994 3496 50  0000 L CNN
-F 1 "DF02M" H 2994 3405 50  0000 L CNN
-F 2 "Diode_THT:Diode_Bridge_DIP-4_W7.62mm_P5.08mm" H 2800 3575 50  0001 L CNN
-F 3 "http://www.vishay.com/docs/88571/dfm.pdf" H 2650 3450 50  0001 C CNN
-	1    2650 3450
-	1    0    0    -1
-$EndComp
-$Comp
-L power:PRI_LO #PWR0123
+L power:PRI_LO #PWR07
 U 1 1 5F363FB3
-P 2650 3950
-F 0 "#PWR0123" H 2650 3800 50  0001 C CNN
-F 1 "PRI_LO" H 2665 4123 50  0000 C CNN
-F 2 "" H 2650 3950 50  0001 C CNN
-F 3 "" H 2650 3950 50  0001 C CNN
-	1    2650 3950
+P 3550 3800
+F 0 "#PWR07" H 3550 3650 50  0001 C CNN
+F 1 "PRI_LO" H 3565 3973 50  0000 C CNN
+F 2 "" H 3550 3800 50  0001 C CNN
+F 3 "" H 3550 3800 50  0001 C CNN
+	1    3550 3800
 	-1   0    0    1
 $EndComp
-Wire Wire Line
-	2650 3000 2650 3150
-Wire Wire Line
-	2650 3750 2650 3950
-Wire Wire Line
-	2100 3450 2350 3450
-Wire Wire Line
-	2950 3450 3350 3450
+$Comp
+L df01s:DF01S CR1
+U 1 1 5FA88EFB
+P 1550 3500
+F 0 "CR1" H 2550 3887 60  0000 C CNN
+F 1 "DF01S" H 2550 3781 60  0000 C CNN
+F 2 "df01s:DF01S" H 2550 3740 60  0001 C CNN
+F 3 "" H 1550 3500 60  0000 C CNN
+	1    1550 3500
+	1    0    0    -1
+$EndComp
+Wire Wire Line
+	1550 3300 1550 3500
+Wire Wire Line
+	1550 3600 1550 3750
+Wire Wire Line
+	3550 3500 3550 3250
+Wire Wire Line
+	3550 3600 3550 3800
 $EndSCHEMATC
