File: Cell/Layout/Processor/Processor.sch (KiCad schematic (older format))
At the start: 6 parts, among them SW1 SW_Push, U1 STM32G030F6P6, U6 SN74LVC1T45DBVR

Commit message: Do the processor board layout
Parts:
- renumbered R2 to R1, R3 to R2, R1 to R3, U6 to U1, U1 to U2
Changed lines of the file:
@@
 $EndDescr
 $Comp
-L stm32g030f6p6:STM32G030F6P6 U1
+L stm32g030f6p6:STM32G030F6P6 U2
 U 1 1 5FA37DB2
 P 4450 2900
-F 0 "U1" H 6250 3387 60  0000 C CNN
+F 0 "U2" H 6250 3387 60  0000 C CNN
 F 1 "STM32G030F6P6" H 6250 3281 60  0000 C CNN
 F 2 "stm32g030f6p6:STM32G030F6P6" H 6250 3240 60  0001 C CNN
@@
 $EndComp
 $Comp
-L Device:R_US R1
+L Device:R_US R3
 U 1 1 5FA5CB7B
 P 4650 1550
-F 0 "R1" H 4718 1596 50  0000 L CNN
+F 0 "R3" H 4718 1596 50  0000 L CNN
 F 1 "R_US" H 4718 1505 50  0000 L CNN
 F 2 "Resistor_SMD:R_0603_1608Metric_Pad1.05x0.95mm_HandSolder" V 4690 1540 50  0001 C CNN
@@
 $EndComp
 $Comp
-L SparkFun-PowerSymbols:3.3V #SUPPLY0101
+L SparkFun-PowerSymbols:3.3V #SUPPLY04
 U 1 1 5FA5D257
 P 4150 3700
-F 0 "#SUPPLY0101" H 4200 3700 45  0001 L BNN
+F 0 "#SUPPLY04" H 4200 3700 45  0001 L BNN
 F 1 "3.3V" H 4150 3976 45  0000 C CNN
 F 2 "XXX-00000" H 4150 3881 60  0000 C CNN
@@
 	4150 3700 4450 3700
 $Comp
-L SparkFun-PowerSymbols:GND #GND0101
+L SparkFun-PowerSymbols:GND #GND05
 U 1 1 5FA5DA03
 P 8050 4400
-F 0 "#GND0101" H 8100 4350 45  0001 L BNN
+F 0 "#GND05" H 8100 4350 45  0001 L BNN
 F 1 "GND" H 8050 4230 45  0000 C CNN
 F 2 "" H 8050 4300 60  0001 C CNN
@@
 	4400 1700 4650 1700
 $Comp
-L SparkFun-PowerSymbols:GND #GND0102
+L SparkFun-PowerSymbols:GND #GND04
 U 1 1 5FA5F842
 P 4000 1850
-F 0 "#GND0102" H 4050 1800 45  0001 L BNN
+F 0 "#GND04" H 4050 1800 45  0001 L BNN
 F 1 "GND" H 4000 1680 45  0000 C CNN
 F 2 "" H 4000 1750 60  0001 C CNN
@@
 	4000 1850 4000 1700
 $Comp
-L SparkFun-PowerSymbols:3.3V #SUPPLY0102
+L SparkFun-PowerSymbols:3.3V #SUPPLY05
 U 1 1 5FA5FC6D
 P 4650 1300
-F 0 "#SUPPLY0102" H 4700 1300 45  0001 L BNN
+F 0 "#SUPPLY05" H 4700 1300 45  0001 L BNN
 F 1 "3.3V" H 4650 1576 45  0000 C CNN
 F 2 "XXX-00000" H 4650 1481 60  0000 C CNN
@@
 SDA
 $Comp
-L Device:R_US R2
+L Device:R_US R1
 U 1 1 5FA83D80
 P 2600 5450
-F 0 "R2" H 2668 5496 50  0000 L CNN
+F 0 "R1" H 2668 5496 50  0000 L CNN
 F 1 "R_US" H 2668 5405 50  0000 L CNN
 F 2 "Resistor_SMD:R_0603_1608Metric_Pad1.05x0.95mm_HandSolder" V 2640 5440 50  0001 C CNN
@@
 $EndComp
 $Comp
-L Device:R_US R3
+L Device:R_US R2
 U 1 1 5FA84CE2
 P 3150 5450
-F 0 "R3" H 3218 5496 50  0000 L CNN
+F 0 "R2" H 3218 5496 50  0000 L CNN
 F 1 "R_US" H 3218 5405 50  0000 L CNN
 F 2 "Resistor_SMD:R_0603_1608Metric_Pad1.05x0.95mm_HandSolder" V 3190 5440 50  0001 C CNN
@@
 	3150 5850 2100 5850
 $Comp
-L SparkFun-PowerSymbols:3.3V #SUPPLY0104
+L SparkFun-PowerSymbols:3.3V #SUPPLY03
 U 1 1 5FA86EA2
 P 3150 5150
-F 0 "#SUPPLY0104" H 3200 5150 45  0001 L BNN
+F 0 "#SUPPLY03" H 3200 5150 45  0001 L BNN
 F 1 "3.3V" H 3150 5426 45  0000 C CNN
 F 2 "XXX-00000" H 3150 5331 60  0000 C CNN
@@
 SDA
 $Comp
-L dk_Logic-Translators-Level-Shifters:SN74LVC1T45DBVR U6
+L dk_Logic-Translators-Level-Shifters:SN74LVC1T45DBVR U1
 U 1 1 5FA4BDE1
 P 2650 3300
-F 0 "U6" H 2994 3353 60  0000 L CNN
+F 0 "U1" H 2994 3353 60  0000 L CNN
 F 1 "SN74LVC1T45DBVR" H 2250 2500 60  0000 L CNN
 F 2 "digikey-footprints:SOT-23-6" H 2850 3500 60  0001 L CNN
@@
 $EndComp
 $Comp
-L SparkFun-PowerSymbols:3.3V #SUPPLY0105
+L SparkFun-PowerSymbols:3.3V #SUPPLY02
 U 1 1 5FA51948
 P 2750 2800
-F 0 "#SUPPLY0105" H 2800 2800 45  0001 L BNN
+F 0 "#SUPPLY02" H 2800 2800 45  0001 L BNN
 F 1 "3.3V" H 2750 3076 45  0000 C CNN
 F 2 "XXX-00000" H 2750 2981 60  0000 C CNN
@@
 $EndComp
 $Comp
-L SparkFun-PowerSymbols:5V #SUPPLY0106
+L SparkFun-PowerSymbols:5V #SUPPLY01
 U 1 1 5FA51F19
 P 2650 2450
-F 0 "#SUPPLY0106" H 2700 2450 45  0001 L BNN
+F 0 "#SUPPLY01" H 2700 2450 45  0001 L BNN
 F 1 "5V" H 2650 2726 45  0000 C CNN
 F 2 "XXX-00000" H 2650 2631 60  0000 C CNN
@@
 $EndComp
 $Comp
-L SparkFun-PowerSymbols:GND #GND0106
+L SparkFun-PowerSymbols:GND #GND03
 U 1 1 5FA53191
 P 2750 3800
-F 0 "#GND0106" H 2800 3750 45  0001 L BNN
+F 0 "#GND03" H 2800 3750 45  0001 L BNN
 F 1 "GND" H 2750 3630 45  0000 C CNN
 F 2 "" H 2750 3700 60  0001 C CNN
